File: pcb/OnionStraws.kicad_sch (KiCad schematic)
At the start: 61 parts, among them J1 Conn_01x04, J2 8P8C, Q1 Si2309CDS, Q2 Si2309CDS, SW1 SW_Push, U1 74LVC2G07, U2 74LVC2G07_3v3, U3 ESP32, U4 APX803L

Commit message: v2 beta
Parts:
- removed C7: 1u, Capacitor_SMD:C_0805_2012Metric, symbol Device:C
- removed J1: Conn_01x04, Connector_PinHeader_2.54mm:PinHeader_1x04_P2.54mm_Horizontal, symbol Connector_Generic:Conn_01x04
- removed R77: 270k, Resistor_SMD:R_0805_2012Metric, symbol Device:R
- removed R88, R99: 10K, Resistor_SMD:R_0805_2012Metric, symbol Device:R
- removed TP3: TestPoint, TestPoint:TestPoint_THTPad_D2.5mm_Drill1.2mm, symbol Connector:TestPoint
- removed U3: ESP32, Library:DIP-38_900_ELL, symbol onionStraws:ESP32
- added C10, C12, C14: 100n, Capacitor_SMD:C_0805_2012Metric, symbol Device:C
- added C13: 10u, Capacitor_SMD:C_0805_2012Metric, symbol Device:C
- added D4: GRN, LED_SMD:LED_0805_2012Metric, symbol Device:LED
- added D5: RED, LED_SMD:LED_0805_2012Metric, symbol Device:LED
- added F1: Polyfuse, Fuse:Fuse_1812_4532Metric, symbol Device:Polyfuse
- added J2: 1x6, Connector_PinHeader_2.54mm:PinHeader_1x06_P2.54mm_Vertical, symbol Connector_Generic:Conn_01x06
- added J3: TC2030, Connector:Tag-Connect_TC2030-IDC-NL_2x03_P1.27mm_Vertical, symbol Connector_Generic:Conn_01x06
- added JP1: FirstBuild, Jumper:SolderJumper-3_P1.3mm_Bridged12_RoundedPad1.0x1.5mm_NumberLabels, symbol Jumper:SolderJumper_3_Bridged12
- added JP2: AltPwr, Jumper:SolderJumper-3_P1.3mm_Bridged12_RoundedPad1.0x1.5mm_NumberLabels, symbol Jumper:SolderJumper_3_Bridged12
- added R1, R2, R3, R5: 10K, Resistor_SMD:R_0805_2012Metric, symbol Device:R
- added R4, R6: 220, Resistor_SMD:R_0805_2012Metric, symbol Device:R
- added SW1: SW_Push, Button_Switch_SMD:SW_Push_1P1T_XKB_TS-1187A, symbol Switch:SW_Push
- added U2: ESP32-C3-WROOM-02, RF_Module:ESP32-C3-WROOM-02, symbol RF_Module:ESP32-C3-WROOM-02
- added U3: L7805, Package_TO_SOT_SMD:TO-263-2, symbol Regulator_Linear:L7805
- added U6: AP2205-3.3, Package_TO_SOT_SMD:SOT-89-3, symbol Regulator_Linear:AP2204R-3.3
- C2: renamed from C10; value 10u -> 1u
- C3: renamed from C1; footprint Capacitor_Tantalum_SMD:CP_EIA-1608-10_AVX-L -> Capacitor_SMD:C_0805_2012Metric
- C5: renamed from C2; footprint Capacitor_Tantalum_SMD:CP_EIA-1608-10_AVX-L -> Capacitor_SMD:C_0805_2012Metric
- C7: renamed from C3; footprint Capacitor_Tantalum_SMD:CP_EIA-1608-10_AVX-L -> Capacitor_SMD:C_0805_2012Metric
- D6: value LED -> YLW; footprint LED_THT:LED_D5.0mm -> LED_SMD:LED_0805_2012Metric
- D8: renamed from D5; footprint Diode_SMD:D_SOD-123 -> Diode_SMD:D_SOD-523
- F2: renamed from F1; footprint Resistor_SMD:R_1210_3225Metric_Pad1.30x2.65mm_HandSolder -> Fuse:Fuse_1812_4532Metric
- H3: now not fitted
- H4: renamed from H2; now not fitted
- R18: renamed from R3; value 270k -> 220k
- R21: renamed from R17; value 270k -> 220k
- R8: renamed from R1; now not fitted
- SW2: renamed from SW1; footprint Button_Switch_THT:SW_PUSH_6mm_H13mm -> Button_Switch_SMD:SW_Push_1P1T_XKB_TS-1187A
- TP1: renamed from TP5; footprint TestPoint:TestPoint_THTPad_D2.5mm_Drill1.2mm -> TestPoint:TestPoint_Pad_D2.0mm; now not fitted
- TP2: renamed from TP7; footprint TestPoint:TestPoint_THTPad_D2.5mm_Drill1.2mm -> TestPoint:TestPoint_Pad_D2.0mm; now not fitted
- TP3: renamed from TP1; footprint TestPoint:TestPoint_THTPad_D2.5mm_Drill1.2mm -> TestPoint:TestPoint_Pad_D2.0mm; now not fitted
- TP4: renamed from TP2; footprint TestPoint:TestPoint_THTPad_D2.5mm_Drill1.2mm -> TestPoint:TestPoint_Pad_D2.0mm; now not fitted
- TP5: renamed from TP4; footprint TestPoint:TestPoint_THTPad_D2.5mm_Drill1.2mm -> TestPoint:TestPoint_Pad_D2.0mm; now not fitted
- TP6: footprint TestPoint:TestPoint_THTPad_D2.5mm_Drill1.2mm -> TestPoint:TestPoint_Pad_D2.0mm; now not fitted
- U1: renamed from U4; value APX803L -> APX803L20-29SA-7
- renumbered C8 to C1, C6 to C11, C11 to C4, C9 to C6, C4 to C8, C5 to C9, D4 to D9, H4 to H2, J2 to J1, R11 to R10, R12 to R11, R14 to R12, R16 to R13, R6 to R14, R7 to R15, R8 to R16, R9 to R17, R10 to R19, R13 to R20, R5 to R22, R4 to R23, R15 to R24, R18 to R25, R19 to R7, R2 to R9, U1 to U4, U2 to U5
Connections:
- net +3V3: now also C6.2, U1.3 (Vcc), C13.1, C14.2, J2.1 (Pin_1), J3.2 (Pin_2), R1.2, R2.1, R3.2, R4.2, R5.2, U2.1 (3V3), U6.3 (VOUT)
- net +5V: now also C12.2, U3.3 (OUT), U6.1 (VIN); no longer C6.2, U1.3 (Vcc)
- net GND: now also C10.1, C12.1, C13.2, C14.1, D4.1 (K), J2.2 (Pin_2), J3.4 (Pin_4), SW1.2, U2.19 (GND), U2.9 (GND), U3.2 (GND), U6.2 (GND)
- net VDC: now also F2.1; no longer F2.2, TP3.1
- net p1: now also TP3.1, JP2.2 (C); no longer F2.1
- net p3: now also C10.2, U3.1 (IN)
- net ALT_PWR: now reaches J1.3
- net ALT_PWR: now also F1.1
- net GEA3_TX: now reaches R13.1
- net GEA3_TX: now also J2.4 (Pin_4), J3.5 (Pin_5), U2.11 (IO20/RXD)
- net LED1: now reaches R7.2
- net LED1: now also U2.3 (IO4)
- net GEA2_RX: now reaches R10.1
- net GEA2_RX: now also U2.10 (IO10)
- net EN: now reaches U1.2 (~{RESET})
- net EN: now also J2.6 (Pin_6), J3.1 (Pin_1), R3.1, U2.2 (EN)
- net BOOT: now reaches SW2.2
- net BOOT: now also J2.3 (Pin_3), J3.6 (Pin_6), JP1.3 (B), R2.2, U2.8 (IO9)
- net GEA3_RX: now reaches R12.1
- net GEA3_RX: now also J2.5 (Pin_5), J3.3 (Pin_3), U2.12 (IO21/TXD)
- net GEA2_TX: now reaches R11.1
- net GEA2_TX: now also JP1.2 (C)
- new net: F2.2, JP2.1 (A)
- new net: D4.2 (A), R6.2
- new net: D5.2 (A), R4.1
- new net: F1.2, JP2.3 (B)
- new net: JP1.1 (A), U2.4 (IO5)
- new net BOOT_SEL: R1.1, SW1.1, U2.7 (IO8)
- new net DBG_LED: D5.1 (K), R5.1, U2.16 (IO2)
- new net LED2: R6.1, U2.15 (IO3)
- no-connect marks 31 -> 9
Other:
- note added: "Tried to be compatible with FirstBuild v1.0 DBG Led ~inverted~ GPIO9 is strapping pin. Pull down by GEA bus could be a problem. JP1 defaults to GPIO5"
- note added: "Voltage Supervisor, Hold ESP reset for 150ms after power reaches 2.9V. Prevent brownout at boot."
- note removed: "EN"
- note removed: "GND"
- note removed: "SMPS Module DC Buck"
- note removed: "VI"
- note removed: "VO"
- note removed: "Voltage Supervisor, Hold ESP reset for 400ms after power reaches 5V. Prevent brownout at boot."
- moved on the sheet: C1, C11, C2, C3, C4, C5, C6, C7, C8, C9, D1, D2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

Commit message: pcb 2.1 mods
Parts:
- removed H3, H4: MountingHole, MountingHole:MountingHole_3.2mm_M3_DIN965, symbol Mechanical:MountingHole
- added TP7: TestPoint, TestPoint:TestPoint_Pad_D2.0mm, symbol Connector:TestPoint
- D8: footprint Diode_SMD:D_SOD-523 -> Diode_SMD:D_SOD-123
Connections:
- net GND: now also TP7.1
Other:
- note added: "2.1 changes Added ground test point Change D8 to bigger part move rj45 inboard 4.5mm smaller 7805 or different ldo"
Changed lines of the file:
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@@
 	)
 	(junction
+		(at 48.26 146.05)
+		(diameter 0)
+		(color 0 0 0 0)
+	)
+	(junction
 		(at 335.915 167.64)
 		(diameter 0)
@@
 	(wire
 		(pts
-			(xy 260.35 43.18) (xy 260.35 50.8)
+			(xy 36.83 146.05) (xy 48.26 146.05)
 		)
 		(stroke
@@
 	(wire
 		(pts
-			(xy 335.915 147.955) (xy 335.915 143.51)
+			(xy 260.35 43.18) (xy 260.35 50.8)
 		)
 		(stroke
@@
 	(wire
 		(pts
-			(xy 149.86 137.16) (xy 149.86 144.78)
+			(xy 335.915 147.955) (xy 335.915 143.51)
 		)
 		(stroke
@@
 	(wire
 		(pts
-			(xy 207.645 54.61) (xy 207.645 57.785)
+			(xy 149.86 137.16) (xy 149.86 144.78)
 		)
 		(stroke
@@
 	(wire
 		(pts
-			(xy 156.21 165.1) (xy 171.45 165.1)
+			(xy 207.645 54.61) (xy 207.645 57.785)
 		)
 		(stroke
@@
 	(wire
 		(pts
-			(xy 289.56 140.97) (xy 289.56 163.83)
+			(xy 156.21 165.1) (xy 171.45 165.1)
 		)
 		(stroke
@@
 	(wire
 		(pts
-			(xy 36.83 147.955) (xy 47.625 147.955)
+			(xy 289.56 140.97) (xy 289.56 163.83)
 		)
 		(stroke
@@
 	(wire
 		(pts
+			(xy 58.42 144.78) (xy 58.42 146.05)
+		)
+		(stroke
+			(width 0)
+			(type default)
+		)
+	)
+	(wire
+		(pts
 			(xy 158.75 134.62) (xy 171.45 134.62)
 		)
@@
 	(wire
 		(pts
-			(xy 47.625 147.955) (xy 47.625 149.86)
+			(xy 48.26 146.05) (xy 48.26 148.59)
 		)
 		(stroke
@@
 	(wire
 		(pts
-			(xy 36.83 144.78) (xy 36.83 147.955)
+			(xy 36.83 144.78) (xy 36.83 146.05)
 		)
 		(stroke
@@
 	(wire
 		(pts
+			(xy 58.42 146.05) (xy 48.26 146.05)
+		)
+		(stroke
+			(width 0)
+			(type default)
+		)
+	)
+	(wire
+		(pts
 			(xy 91.44 36.83) (xy 95.25 36.83)
 		)
@@
 	)
 	(image
-		(at 254 231.14)
+		(at 254.254 312.928)
 		(scale 0.319381)
 		(data "iVBORw0KGgoAAAANSUhEUgAADjsAAAe0CAIAAAAycNZhAAAAA3NCSVQICAjb4U/gAAAgAElEQVR4"
@@
 		)
 	)
+	(text "2.1 changes\n\nAdded ground test point\nChange D8 to bigger part\n\nmove  rj45 inboard 4.5mm\nsmaller 7805 or different ldo"
+		(exclude_from_sim no)
+		(at 402.844 248.412 0)
+		(effects
+			(font
+				(size 1.27 1.27)
+			)
+		)
+	)
 	(text "Washer\nGND\nNC\nHvoltage side\nRX/TX\nRX/TX\n+5V\nNC\n+16.2V"
 		(exclude_from_sim no)
@@
 	)
 	(symbol
-		(lib_id "Mechanical:MountingHole")
-		(at 159.385 249.555 0)
-		(unit 1)
-		(exclude_from_sim no)
-		(in_bom yes)
-		(on_board yes)
-		(dnp yes)
-		(fields_autoplaced yes)
-		(property "Reference" "H3"
-			(at 161.925 248.6465 0)
-			(effects
-				(font
-					(size 1.27 1.27)
-				)
-				(justify left)
-			)
-		)
-		(property "Value" "MountingHole"
-			(at 161.925 251.4216 0)
-			(effects
-				(font
-					(size 1.27 1.27)
-				)
-				(justify left)
-			)
-		)
-		(property "Footprint" "MountingHole:MountingHole_3.2mm_M3_DIN965"
-			(at 159.385 249.555 0)
-			(effects
-				(font
-					(size 1.27 1.27)
-				)
-				(hide yes)
-			)
-		)
-		(property "Datasheet" "~"
-			(at 159.385 249.555 0)
-			(effects
-				(font
-					(size 1.27 1.27)
-				)
-				(hide yes)
-			)
-		)
-		(property "Description" ""
-			(at 159.385 249.555 0)
-			(effects
-				(font
-					(size 1.27 1.27)
-				)
-				(hide yes)
-			)
-		)
-		(instances
-			(project ""
-				(path "/477311b9-8f81-40c8-9c55-fd87e287247a"
-					(reference "H3")
-					(unit 1)
-				)
-			)
-		)
-	)
-	(symbol
 		(lib_id "Device:C")
 		(at 260.35 54.61 180)
@@
 	(symbol
 		(lib_id "power:GND")
-		(at 47.625 149.86 0)
+		(at 48.26 148.59 0)
 		(unit 1)
 		(exclude_from_sim no)
@@
 		(fields_autoplaced yes)
 		(property "Reference" "#PWR08"
-			(at 47.625 156.21 0)
+			(at 48.26 154.94 0)
 			(effects
 				(font
@@
 		)
 		(property "Value" "GND"
-			(at 47.625 154.4225 0)
+			(at 48.26 153.1525 0)
 			(effects
 				(font
@@
 		)
 		(property "Footprint" ""
-			(at 47.625 149.86 0)
+			(at 48.26 148.59 0)
 			(effects
 				(font
@@
 		)
 		(property "Datasheet" ""
-			(at 47.625 149.86 0)
+			(at 48.26 148.59 0)
 			(effects
 				(font
@@
 		)
 		(property "Description" ""
-			(at 47.625 149.86 0)
+			(at 48.26 148.59 0)
 			(effects
 				(font
@@
 	)
 	(symbol
+		(lib_id "Connector:TestPoint")
+		(at 58.42 144.78 0)
+		(unit 1)
+		(exclude_from_sim no)
+		(in_bom yes)
+		(on_board yes)
+		(dnp yes)
+		(fields_autoplaced yes)
+		(property "Reference" "TP7"
+			(at 59.817 140.5695 0)
+			(effects
+				(font
+					(size 1.27 1.27)
+				)
+				(justify left)
+			)
+		)
+		(property "Value" "TestPoint"
+			(at 59.817 143.3446 0)
+			(effects
+				(font
+					(size 1.27 1.27)
+				)
+				(justify left)
+			)
+		)
+		(property "Footprint" "TestPoint:TestPoint_Pad_D2.0mm"
+			(at 63.5 144.78 0)
+			(effects
+				(font
+					(size 1.27 1.27)
+				)
+				(hide yes)
+			)
+		)
+		(property "Datasheet" "~"
+			(at 63.5 144.78 0)
+			(effects
+				(font
+					(size 1.27 1.27)
+				)
+				(hide yes)
+			)
+		)
+		(property "Description" ""
+			(at 58.42 144.78 0)
+			(effects
+				(font
+					(size 1.27 1.27)
+				)
+				(hide yes)
+			)
+		)
+		(pin "1"
+		)
+		(instances
+			(project "OnionStraws"
+				(path "/477311b9-8f81-40c8-9c55-fd87e287247a"
+					(reference "TP7")
+					(unit 1)
+				)
+			)
+		)
+	)
+	(symbol
 		(lib_id "power:GND")
 		(at 320.675 150.495 0)
@@
 			)
 		)
-		(property "Footprint" "Diode_SMD:D_SOD-523"
+		(property "Footprint" "Diode_SMD:D_SOD-123"
 			(at 289.56 55.88 0)
 			(effects
@@
 			)
 		)
-		(property "Description" "C2993047"
+		(property "Description" "C78479"
 			(at 289.56 55.88 0)
 			(effects
@@
 					(unit 1)
 				)
-			)
-		)
-	)
-	(symbol
-		(lib_id "Mechanical:MountingHole")
-		(at 160.02 242.57 0)
-		(unit 1)
-		(exclude_from_sim no)
-		(in_bom yes)
-		(on_board yes)
-		(dnp yes)
-		(fields_autoplaced yes)
-		(property "Reference" "H4"
-			(at 162.56 241.6615 0)
-			(effects
-				(font
-					(size 1.27 1.27)
-				)
-				(justify left)
-			)
-		)
-		(property "Value" "MountingHole"
-			(at 162.56 244.4366 0)
-			(effects
-				(font
-					(size 1.27 1.27)
-				)
-				(justify left)
-			)
-		)
-		(property "Footprint" "MountingHole:MountingHole_3.2mm_M3_DIN965"
-			(at 160.02 242.57 0)
-			(effects
-				(font
-					(size 1.27 1.27)
-				)
-				(hide yes)
-			)
-		)
-		(property "Datasheet" "~"
-			(at 160.02 242.57 0)
-			(effects
-				(font
-					(size 1.27 1.27)
-				)
-				(hide yes)
-			)
-		)
-		(property "Description" ""
-			(at 160.02 242.57 0)
-			(effects
-				(font
-					(size 1.27 1.27)
-				)
-				(hide yes)
-			)
-		)
-		(instances
-			(project ""
-				(path "/477311b9-8f81-40c8-9c55-fd87e287247a"
-					(reference "H4")
-					(unit 1)
-				)
